Commit message: Update omni_description

File: rmcs_ws/src/omni_description/urdf/omni_description.urdf (robot description, URDF)
Before this commit: robot urdf.SLDASM, 10 links, 9 joints
Links:
- removed link Total assembly
- removed link back left wheel
- removed link back right wheel
- removed link body&gimbol
- removed link body&wheels
- removed link frout left wheel
- removed link frout right wheel
- removed link gimbol
- removed link gimbol&launch
- removed link launch
- added link back_left_wheel, mass 0.533176182602155; collision mesh filename=package://omni_description/meshes/back_left_wheel.STL; visual mesh filename=package://omni_description/meshes/back_left_wheel.STL
- added link back_right_wheel, mass 0.533176182602155; collision mesh filename=package://omni_description/meshes/back_right_wheel.STL; visual mesh filename=package://omni_description/meshes/back_right_wheel.STL
- added link body, mass 7.38762341423434; collision mesh filename=package://omni_description/meshes/body.STL; visual mesh filename=package://omni_description/meshes/body.STL
- added link front_left_wheel, mass 0.533176182602155; collision mesh filename=package://omni_description/meshes/front_left_wheel.STL; visual mesh filename=package://omni_description/meshes/front_left_wheel.STL
- added link front_right_wheel, mass 0.533176182602155; collision mesh filename=package://omni_description/meshes/front_right_wheel.STL; visual mesh filename=package://omni_description/meshes/front_right_wheel.STL
- added link gimbol_pitch, mass 2.85600268929187; collision mesh filename=package://omni_description/meshes/gimbol_pitch.STL; visual mesh filename=package://omni_description/meshes/gimbol_pitch.STL
- added link gimbol_yaw, mass 0.296006965244182; collision mesh filename=package://omni_description/meshes/gimbol_yaw.STL; visual mesh filename=package://omni_description/meshes/gimbol_yaw.STL
- added link left_launch, mass 0.0265195187658292; collision mesh filename=package://omni_description/meshes/left_launch.STL; visual mesh filename=package://omni_description/meshes/left_launch.STL
- added link omni_description, mass 12.7253768367107; collision mesh filename=package://omni_description/meshes/omni_description.STL; visual mesh filename=package://omni_description/meshes/omni_description.STL
- added link right_launch, mass 0.0265195187658292; collision mesh filename=package://omni_description/meshes/right_launch.STL; visual mesh filename=package://omni_description/meshes/right_launch.STL
Joints:
- removed joint back left wheel
- removed joint back right wheel
- removed joint body&gimbol
- removed joint body&wheels
- removed joint frout left wheel
- removed joint frout right wheel
- removed joint gimbol
- removed joint gimbol&launch
- removed joint launch
- added joint back_left_wheel: type revolute, parent body, child back_left_wheel, origin xyz=-0.13409 0.1955 -0.28694 rpy=0.25256 -0.050385 1.7635, axis -1 0 0, limit lower=0 upper=0 effort=0 velocity=0
- added joint back_right_wheel: type revolute, parent body, child back_right_wheel, origin xyz=-0.31291 -0.08302 -0.23959 rpy=-0.052033 -0.25223 -2.9359, axis -1 0 0, limit lower=0 upper=0 effort=0 velocity=0
- added joint body: type fixed, parent omni_description, child body, origin xyz=-0.0118523156712267 0.0356448860509371 0.220657130432317 rpy=0 -0.257427286657566 0.586263535297581, axis 0 0 0
- added joint front_left_wheel: type revolute, parent body, child front_left_wheel, origin xyz=0.13532 0.01052 -0.35759 rpy=0.052033 0.25223 0.20573, axis 1 0 0, limit lower=0 upper=0 effort=0 velocity=0
- added joint front_right_wheel: type revolute, parent body, child front_right_wheel, origin xyz=-0.043633 -0.268 -0.31076 rpy=-0.25256 0.050385 -1.3781, axis 1 0 0, limit lower=0 upper=0 effort=0 velocity=0
- added joint gimbol_pitch: type revolute, parent gimbol_yaw, child gimbol_pitch, origin xyz=0 0 0.0934 rpy=0 -0.25743 0, axis 0 -1 0, limit lower=0 upper=0 effort=0 velocity=0
- added joint gimbol_yaw: type revolute, parent body, child gimbol_yaw, origin xyz=-0.036779 -0.03625 -0.10102 rpy=0 0.25743 0, axis 0 0 -1, limit lower=0 upper=0 effort=0 velocity=0
- added joint left_launch: type revolute, parent gimbol_pitch, child left_launch, origin xyz=0.013 0.03625 0.0107 rpy=0 0 0, axis 0 0 -1, limit lower=0 upper=0 effort=0 velocity=0
- added joint right_launch: type revolute, parent gimbol_pitch, child right_launch, origin xyz=0.013 -0.03625 0.0107 rpy=0 0 0, axis 0 0 -1, limit lower=0 upper=0 effort=0 velocity=0
