Commit message: Add chasis controller

File: rmcs_ws/src/omni_infantry_description/urdf/omni_infantry/omni_infantry_macro.ros2_control.xacro (robot description, xacro)
@@ -63,5 +63,5 @@
         <state_interface name="velocity" />
       </joint>
-      <joint name="${prefix}yaw">
+      <!-- <joint name="${prefix}yaw">
         <command_interface name="effort">
           <param name="min">-16384</param>
@@ -94,5 +94,5 @@
         <state_interface name="position" />
         <state_interface name="velocity" />
-      </joint>
+      </joint> -->
     </ros2_control>
     <xacro:if value="$(arg sim_gazebo_classic)">
