Commit message: Update omni_infantry_description package

File: rmcs_ws/src/omni_infantry_description/urdf/omni_infantry.urdf.xacro (robot description, xacro)
@@ -9,14 +9,7 @@
   <xacro:arg name="simulation_controllers" default="" />
   <xacro:include
-    filename="$(find omni_infantry_description)/urdf/omni_infantry/omni_infantry_macro.xacro" />
+    filename="$(find omni_infantry_description)/urdf/omni_infantry/omni_infantry_description.urdf" />
   <xacro:include
     filename="$(find omni_infantry_description)/urdf/omni_infantry/omni_infantry_macro.ros2_control.xacro" />
-  <!-- create link fixed to the "world" -->
-  <link name="world" />
-  <!-- Load robot's macro with parameters -->
-  <!-- set prefix if multiple robots are used -->
-  <xacro:omni_infantry prefix="$(arg prefix)" parent="world">
-    <origin xyz="0 0 0" rpy="0 0 0" />          <!-- position robot in the world -->
-  </xacro:omni_infantry>
   <xacro:omni_infantry_ros2_control
     name="omni_infantry"

File: rmcs_ws/src/omni_infantry_description/urdf/omni_infantry/omni_infantry_description.urdf (robot description, URDF)
Before this commit: robot omni_description, 10 links, 9 joints
Links:
- link back_left_wheel: geometry collision mesh filename=package://omni_infantry_description/meshes/back_left_wheel.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; visual mesh filename=package://omni_infantry_description/meshes/back_left_wheel.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
- link back_right_wheel: geometry collision mesh filename=package://omni_infantry_description/meshes/back_right_wheel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; visual mesh filename=package://omni_infantry_description/meshes/back_right_wheel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
- link body: geometry collision mesh filename=package://omni_infantry_description/meshes/body.STL; visual mesh filename=package://omni_infantry_description/meshes/body.STL
- link front_left_wheel: geometry collision mesh filename=package://omni_infantry_description/meshes/front_left_wheel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; visual mesh filename=package://omni_infantry_description/meshes/front_left_wheel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
- link front_right_wheel: geometry collision mesh filename=package://omni_infantry_description/meshes/front_right_whee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; visual mesh filename=package://omni_infantry_description/meshes/front_right_whee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
- link gimbol_pitch: geometry collision mesh filename=package://omni_infantry_description/meshes/gimbol_pitch.STL; visual mesh filename=package://omni_infantry_description/meshes/gimbol_pitch.STL
- link gimbol_yaw: geometry collision mesh filename=package://omni_infantry_description/meshes/gimbol_yaw.STL; visual mesh filename=package://omni_infantry_description/meshes/gimbol_yaw.STL
- link left_launch: geometry collision mesh filename=package://omni_infantry_description/meshes/left_launch.STL; visual mesh filename=package://omni_infantry_description/meshes/left_launch.STL
- link omni_description: geometry collision mesh filename=package://omni_infantry_description/meshes/omni_description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; visual mesh filename=package://omni_infantry_description/meshes/omni_description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
- link right_launch: geometry collision mesh filename=package://omni_infantry_description/meshes/right_launch.STL; visual mesh filename=package://omni_infantry_description/meshes/right_launch.STL
Joints:
- joint back_left_wheel: type revolute -> continuous
- joint back_right_wheel: type revolute -> continuous
- joint front_left_wheel: type revolute -> continuous
- joint front_right_wheel: type revolute -> continuous
- joint gimbol_yaw: type revolute -> continuous
- joint left_launch: type revolute -> continuous
- joint right_launch: type revolute -> continuous

File: rmcs_ws/src/omni_infantry_description/urdf/omni_infantry/omni_infantry_macro.ros2_control.xacro (robot description, xacro)
@@ -30,91 +30,37 @@
         </xacro:unless>
       </hardware>
-      <joint name="${prefix}joint1">
-        <command_interface name="position">     <!-- Add/Remove interfaces as needed -->
-          <param name="min">-1</param>
-          <param name="max">1</param>
+      <!-- Motor type  RoboMaster 3508 -->
+      <joint name="${prefix}front_left_wheel">
+        <command_interface name="effort">
+          <param name="min">-16384</param>
+          <param name="max">16384</param>
         </command_interface>
-        <state_interface name="position">
-          <param name="initial_value">0.0</param>
-        </state_interface>
+        <state_interface name="position" />
         <state_interface name="velocity" />
-        <state_interface name="acceleration" />
       </joint>
-      <joint name="${prefix}joint2">
-        <command_interface name="position">     <!-- Add/Remove interfaces as needed -->
-          <param name="min">-1</param>
-          <param name="max">1</param>
+      <joint name="${prefix}front_right_wheel">
+        <command_interface name="effort">
+          <param name="min">-16384</param>
+          <param name="max">16384</param>
         </command_interface>
-        <state_interface name="position">
-          <param name="initial_value">0.0</param>
-        </state_interface>
+        <state_interface name="position" />
         <state_interface name="velocity" />
-        <state_interface name="acceleration" />
       </joint>
-      <joint name="${prefix}joint3">
-        <command_interface name="position">     <!-- Add/Remove interfaces as needed -->
-          <param name="min">-1</param>
-          <param name="max">1</param>
+      <joint name="${prefix}back_left_wheel">
+        <command_interface name="effort">
+          <param name="min">-16384</param>
+          <param name="max">16384</param>
         </command_interface>
-        <state_interface name="position">
-          <param name="initial_value">0.0</param>
-        </state_interface>
+        <state_interface name="position" />
         <state_interface name="velocity" />
-        <state_interface name="acceleration" />
       </joint>
-      <joint name="${prefix}joint4">
-        <command_interface name="position">     <!-- Add/Remove interfaces as needed -->
-          <param name="min">-1</param>
-          <param name="max">1</param>
+      <joint name="${prefix}back_right_wheel">
+        <command_interface name="effort">
+          <param name="min">-16384</param>
+          <param name="max">16384</param>
         </command_interface>
-        <state_interface name="position">
-          <param name="initial_value">0.0</param>
-        </state_interface>
+        <state_interface name="position" />
         <state_interface name="velocity" />
-        <state_interface name="acceleration" />
       </joint>
-      <joint name="${prefix}joint5">
-        <command_interface name="position">     <!-- Add/Remove interfaces as needed -->
-          <param name="min">-1</param>
-          <param name="max">1</param>
-        </command_interface>
-        <state_interface name="position">
-          <param name="initial_value">0.0</param>
-        </state_interface>
-        <state_interface name="velocity" />
-        <state_interface name="acceleration" />
-      </joint>
-      <joint name="${prefix}joint6">
-        <command_interface name="position">     <!-- Add/Remove interfaces as needed -->
-          <param name="min">-1</param>
-          <param name="max">1</param>
-        </command_interface>
-        <state_interface name="position">
-          <param name="initial_value">0.0</param>
-        </state_interface>
-        <state_interface name="velocity" />
-        <state_interface name="acceleration" />
-      </joint>
-      <sensor name="tcp_fts_sensor">            <!-- Remove/change sensors as needed -->
-        <state_interface name="fx" />
-        <state_interface name="fy" />
-        <state_interface name="fz" />
-        <state_interface name="tx" />
-        <state_interface name="ty" />
-        <state_interface name="tz" />
-        <param name="frame_id">tool0</param>    <!-- Change sensors as needed -->
-        <param name="min_fx">-100</param>
-        <param name="max_fx">100</param>
-        <param name="min_fy">-100</param>
-        <param name="max_fy">100</param>
-        <param name="min_fz">-200</param>
-        <param name="max_fz">200</param>
-        <param name="min_tx">-10</param>
-        <param name="max_tx">10</param>
-        <param name="min_ty">-10</param>
-        <param name="max_ty">10</param>
-        <param name="min_tz">-15</param>
-        <param name="max_tz">15</param>
-      </sensor>
     </ros2_control>
     <xacro:if value="$(arg sim_gazebo_classic)">

Commit message: Update urdf to xacro

File: rmcs_ws/src/omni_infantry_description/urdf/omni_infantry.urdf.xacro (robot description, xacro)
@@ -9,7 +9,11 @@
   <xacro:arg name="simulation_controllers" default="" />
   <xacro:include
-    filename="$(find omni_infantry_description)/urdf/omni_infantry/omni_infantry_description.urdf" />
+    filename="$(find omni_infantry_description)/urdf/omni_infantry/omni_infantry_description.xacro" />
   <xacro:include
     filename="$(find omni_infantry_description)/urdf/omni_infantry/omni_infantry_macro.ros2_control.xacro" />
+  <link name="world" />
+  <xacro:omni_infantry prefix="$(arg prefix)" parent="world">
+    <origin xyz="0 0 0" rpy="0 0 0" />
+  </xacro:omni_infantry>
   <xacro:omni_infantry_ros2_control
     name="omni_infantry"

Commit message: Update description xacro

File: rmcs_ws/src/omni_infantry_description/urdf/omni_infantry.urdf.xacro (robot description, xacro)
@@ -14,5 +14,5 @@
   <link name="world" />
   <xacro:omni_infantry prefix="$(arg prefix)" parent="world">
-    <origin xyz="0 0 0" rpy="0 0 0" />
+    <origin xyz="0 0 0.17" rpy="0 0 0" />
   </xacro:omni_infantry>
   <xacro:omni_infantry_ros2_control

File: rmcs_ws/src/omni_infantry_description/urdf/omni_infantry/omni_infantry_description.xacro (robot description, xacro)
@@ -4,5 +4,4 @@
   <xacro:macro name="omni_infantry" params="prefix parent *origin">
     <!-- LINKS -->
-    <!-- base link -->
     <link name="${prefix}omni_infantry">
       <inertial>
@@ -22,5 +21,5 @@
         <origin
           xyz="0 0 0"
-          rpy="0 0 0" />
+          rpy="-1.570796326794896 0 0" />
         <geometry>
           <mesh filename="package://omni_infantry_description/meshes/omni_infantry.STL" />
@@ -33,5 +32,5 @@
         <origin
           xyz="0 0 0"
-          rpy="0 0 0" />
+          rpy="-1.570796326794896 0 0" />
         <geometry>
           <mesh filename="package://omni_infantry_description/meshes/omni_infantry.STL" />
@@ -193,5 +192,5 @@
         <origin
           xyz="0 0 0"
-          rpy="0 0 0" />
+          rpy="-1.570796326794896 0 0" />
         <geometry>
           <mesh filename="package://omni_infantry_description/meshes/yaw_link.STL" />
@@ -204,5 +203,5 @@
         <origin
           xyz="0 0 0"
-          rpy="0 0 0" />
+          rpy="-1.570796326794896 0 0" />
         <geometry>
           <mesh filename="package://omni_infantry_description/meshes/yaw_link.STL" />
@@ -227,5 +226,5 @@
         <origin
           xyz="0 0 0"
-          rpy="0 0 0" />
+          rpy="-1.570796326794896 0 0" />
         <geometry>
           <mesh filename="package://omni_infantry_description/meshes/pitch_link.STL" />
@@ -238,5 +237,5 @@
         <origin
           xyz="0 0 0"
-          rpy="0 0 0" />
+          rpy="-1.570796326794896 0 0" />
         <geometry>
           <mesh filename="package://omni_infantry_description/meshes/pitch_link.STL" />
@@ -313,5 +312,5 @@
     </link>
     <!-- END LINKS -->
-    <joint name="${prefix}base_joint" type="fixed">
+    <joint name="${prefix}omni_infantry_base" type="fixed">
       <xacro:insert_block name="origin" />
       <parent link="${parent}" />
@@ -366,6 +365,6 @@
       <axis xyz="0 -1 0" />
       <limit
-        lower="-3.14"
-        upper="3.14"
+        lower="-1"
+        upper="0.7"
         effort="0"
         velocity="0" />
