Commit message: Emergency debugging

File: rmcs_ws/src/rmcs_description/urdf/medium_feed_omni_wheel.xacro (robot description, xacro)
@@ -73,3 +73,9 @@
     <origin xyz="0.06603 0 0.082" />
   </joint>
+  <link name="lidar_link" />
+  <joint name="lidar" type="fixed">
+    <parent link="yaw_link" />
+    <child link="lidar_link" />
+    <origin rpy="${pi} 0 ${pi}" xyz="0 0 0.4" />
+  </joint>
 </robot>

Commit message: Adapt rmcs_auto_aim

File: rmcs_ws/src/rmcs_description/urdf/medium_feed_omni_wheel.xacro (robot description, xacro)
@@ -59,5 +59,5 @@
     <parent link="pitch_link" />
     <child link="imu_link" />
-    <origin rpy = "0 0 ${pi/2}" xyz="0 0 0" />
+    <origin rpy="0 0 ${pi/2}" xyz="0 0 0" />
   </joint>
   <link name="muzzle_link" />
@@ -73,3 +73,27 @@
     <origin xyz="0.06603 0 0.082" />
   </joint>
+  <link name="omni_link_left_front" />
+  <joint name="omni" type="fixed">
+    <parent link="yaw_link" />
+    <child link="omni_link_left_front" />
+    <origin xyz="" />
+  </joint>
+  <link name="omni_link_right_front" />
+  <joint name="omni" type="fixed">
+    <parent link="yaw_link" />
+    <child link="omni_link_right_front" />
+    <origin xyz="" />
+  </joint>
+  <link name="omni_link_left" />
+  <joint name="omni" type="fixed">
+    <parent link="yaw_link" />
+    <child link="omni_link_left" />
+    <origin xyz="" />
+  </joint>
+  <link name="omni_link_right" />
+  <joint name="omni" type="fixed">
+    <parent link="yaw_link" />
+    <child link="omni_link_right" />
+    <origin xyz="" />
+  </joint>
 </robot>

Commit message: fix(PowerController):Temp push for ubuntu work

File: rmcs_ws/src/rmcs_description/urdf/medium_feed_omni_wheel.xacro (robot description, xacro)
@@ -59,5 +59,5 @@
     <parent link="pitch_link" />
     <child link="imu_link" />
-    <origin rpy="0 0 ${pi/2}" xyz="0 0 0" />
+    <origin rpy = "0 0 ${pi/2}" xyz="0 0 0" />
   </joint>
   <link name="muzzle_link" />
