Commit message: refactor: simplify link update logic in ArmConfig

File: rmcs_ws/src/arm_description/urdf/arm_description.urdf (robot description, URDF)
Before this commit: robot arm_description, 7 links, 6 joints
Joints:
- joint joint_3: limit lower=-1.2217 upper=0.5235 effort=35 velocity=4.71 -> lower=-1.36217 upper=0.5335 effort=35 velocity=4.71

File: rmcs_ws/src/arm_moveit_config/config/arm_description.urdf.xacro (robot description, xacro)
@@ -1,5 +1,5 @@
 <?xml version="1.0"?>
 <robot xmlns:xacro="http://www.ros.org/wiki/xacro" name="arm_description">
-    <xacro:arg name="initial_positions_file" default="initial_positions.yaml" />
+    <xacro:arg name="initial_positions_file" default="$(find arm_moveit_config)/config/initial_positions.yaml" />
     <!-- Import arm_description urdf file -->
     <xacro:include filename="$(find arm_description)/urdf/arm_description.urdf" />

Commit message: complete moveit_config & arm_config,and refactor frame

File: rmcs_ws/src/arm_description/urdf/arm_description.urdf (robot description, URDF)
Before this commit: robot arm_description, 7 links, 6 joints
Joints:
- joint joint_6: origin xyz=-0.002 0.119 0 rpy=1.5708 0 0 -> xyz=0.0 0.119 0 rpy=1.5708 0 0

Commit message: feat: complete theoretical validation of gravity compensation

File: rmcs_ws/src/arm_description/urdf/arm_description.urdf (robot description, URDF)
Before this commit: robot arm_description, 7 links, 6 joints
Links:
- link link_2: mass 0.292 -> 0.302
- link link_3: mass 1.321 -> 1.721
- link link_4: mass 0.71 -> 1.41
- link link_5: mass 0.324 -> 0.624
- link link_6: mass 0.14108 -> 0.77108
Joints:
- joint joint_5: axis 0 0 -1 -> 0 0 1

Commit message: feat(control): implement friction compensation with improved behavior

File: rmcs_ws/src/arm_description/urdf/arm_description.urdf (robot description, URDF)
Before this commit: robot arm_description, 7 links, 6 joints
Links:
- link link_2: mass 0.302 -> 0.1502
- link link_3: mass 1.721 -> 1.821
- link link_4: mass 1.41 -> 1.61

Commit message: Update：Initial integration with moveit2

File: rmcs_ws/src/arm_description/urdf/arm_description.urdf (robot description, URDF)
Before this commit: robot arm_description, 7 links, 6 joints
Joints:
- joint joint_2: limit lower=-1.047 upper=1.396 effort=63 velocity=4.71 -> lower=-1.084 upper=1.426 effort=63 velocity=4.71
- joint joint_5: axis 0 0 1 -> 0 0 -1

File: rmcs_ws/src/arm_moveit_config/config/arm_description.urdf.xacro (robot description, xacro)
@@ -6,4 +6,4 @@
     <!-- Import control_xacro-->
     <xacro:include filename="arm_description.ros2_control.xacro" />
-    <xacro:arm_description_ros2_control name="FakeSystem" initial_positions_file="$(arg initial_positions_file)"/>
+    <!-- <xacro:arm_description_ros2_control name="FakeSystem" initial_positions_file="$(arg initial_positions_file)"/>  -->
 </robot>

Commit message: save

File: rmcs_ws/src/arm_description/urdf/arm_description.urdf (robot description, URDF)
Before this commit: robot arm_description, 7 links, 6 joints
Links:
- link base_link: mass None -> 0.402123859659494
- link link_1: mass 0.536 -> 0.25868
- link link_2: mass 0.1502 -> 0.18736
- link link_3: mass 1.821 -> 0.42456
- link link_4: mass 1.61 -> 0.25332
- link link_5: mass 0.624 -> 0.080964
- link link_6: mass 0.77108 -> 0.011935
Joints:
- joint joint_1: limit lower=-3.1 upper=3.1 effort=25 velocity=7.75 -> lower=-3 upper=3 effort=30 velocity=5
- joint joint_2: axis 0 0 -1 -> 0 0 1; limit lower=-1.084 upper=1.426 effort=63 velocity=4.71 -> lower=-1.5 upper=1.5 effort=35 velocity=5; origin xyz=0 -0.042 0.071 rpy=1.5708 0 -3.1416 -> xyz=0 -0.042 0.071 rpy=1.5708 0 0
- joint joint_3: axis 0 0 -1 -> 0 0 1; limit lower=-1.36217 upper=0.5335 effort=35 velocity=4.71 -> lower=-0.8 upper=0.5 effort=35 velocity=5; origin xyz=0 0.37 0.007 rpy=0 0 1.5708 -> xyz=0 0.37 -0.007 rpy=0 0 1.5708
- joint joint_4: limit lower=-3.14 upper=3.14 effort=18 velocity=7.54 -> lower=-3.14 upper=3.14 effort=20 velocity=5; origin xyz=0.03 0.1419 0.035 rpy=-1.5708 0 0 -> xyz=0.03 -0.1419 -0.035 rpy=1.5708 0 0
- joint joint_5: limit lower=-1.74 upper=1.74 effort=6 velocity=24.61 -> lower=-1.3 upper=1.3 effort=10 velocity=5
- joint joint_6: limit lower=-3.14 upper=3.14 effort=3 velocity=10 -> lower=-2.9 upper=2.9 effort=4 velocity=5; origin xyz=0.0 0.119 0 rpy=1.5708 0 0 -> xyz=0 0.026 0 rpy=1.5708 0 0

File: rmcs_ws/src/arm_moveit_config/config/arm_description.urdf.xacro (robot description, xacro)
@@ -1,9 +1,9 @@
 <?xml version="1.0"?>
 <robot xmlns:xacro="http://www.ros.org/wiki/xacro" name="arm_description">
-    <xacro:arg name="initial_positions_file" default="$(find arm_moveit_config)/config/initial_positions.yaml" />
+    <xacro:arg name="initial_positions_file" default="initial_positions.yaml" />
     <!-- Import arm_description urdf file -->
     <xacro:include filename="$(find arm_description)/urdf/arm_description.urdf" />
-    <!-- Import control_xacro-->
+    <!-- Import control_xacro -->
     <xacro:include filename="arm_description.ros2_control.xacro" />
-    <!-- <xacro:arm_description_ros2_control name="FakeSystem" initial_positions_file="$(arg initial_positions_file)"/>  -->
+    <xacro:arm_description_ros2_control name="FakeSystem" initial_positions_file="$(arg initial_positions_file)"/>
 </robot>

Commit message: update

File: rmcs_ws/src/arm_description/urdf/arm_description.urdf (robot description, URDF)
Before this commit: robot arm_description, 7 links, 6 joints
Links:
- link base_link: mass 0.402123859659494 -> 0.079
- link link_1: mass 0.25868 -> 0.743; geometry collision mesh filename=package://arm_description/meshes/Link1.STL; visual mesh filename=package://arm_description/meshes/Link1.STL
- link link_2: mass 0.18736 -> 0.396; geometry collision mesh filename=package://arm_description/meshes/Link2.STL; visual mesh filename=package://arm_description/meshes/Link2.STL
- link link_3: mass 0.42456 -> 0.207; geometry collision mesh filename=package://arm_description/meshes/Link3.STL; visual mesh filename=package://arm_description/meshes/Link3.STL
- link link_4: mass 0.25332 -> 0.371; geometry collision mesh filename=package://arm_description/meshes/Link4.STL; visual mesh filename=package://arm_description/meshes/Link4.STL
- link link_5: mass 0.080964 -> 0.137; geometry collision mesh filename=package://arm_description/meshes/Link5.STL; visual mesh filename=package://arm_description/meshes/Link5.STL
- link link_6: mass 0.011935 -> 0.185; geometry collision mesh filename=package://arm_description/meshes/Link6.STL; visual mesh filename=package://arm_description/meshes/Link6.STL
Joints:
- joint joint_1: limit lower=-3 upper=3 effort=30 velocity=5 -> lower=-3.1 upper=3.1 effort=25 velocity=7.75; origin xyz=0 0 0 rpy=0 0 0 -> xyz=0 0 0.0465 rpy=0 0 0
- joint joint_2: axis 0 0 1 -> 0 0 -1; limit lower=-1.5 upper=1.5 effort=35 velocity=5 -> lower=-1.084 upper=1.426 effort=63 velocity=4.71; origin xyz=0 -0.042 0.071 rpy=1.5708 0 0 -> xyz=0 0 0.0354 rpy=1.5708 0 3.1416
- joint joint_3: axis 0 0 1 -> 0 0 -1; limit lower=-0.8 upper=0.5 effort=35 velocity=5 -> lower=-1.36217 upper=0.5335 effort=35 velocity=4.71; origin xyz=0 0.37 -0.007 rpy=0 0 1.5708 -> xyz=0 0.17331 0 rpy=0 0 1.5708
- joint joint_4: limit lower=-3.14 upper=3.14 effort=20 velocity=5 -> lower=-3.14 upper=3.14 effort=18 velocity=7.54; origin xyz=0.03 -0.1419 -0.035 rpy=1.5708 0 0 -> xyz=0.019039 0.092852 -0.01035 rpy=-1.5708 0 0
- joint joint_5: limit lower=-1.3 upper=1.3 effort=10 velocity=5 -> lower=-1.74 upper=1.74 effort=6 velocity=24.61; origin xyz=0 0 0.2591 rpy=1.5708 0 0 -> xyz=0 0 0.11484 rpy=1.5708 0 0
- joint joint_6: limit lower=-2.9 upper=2.9 effort=4 velocity=5 -> lower=-3.14 upper=3.14 effort=3 velocity=10; origin xyz=0 0.026 0 rpy=1.5708 0 0 -> xyz=0 0.0739 0 rpy=1.5708 0 0

Commit message: 111

File: rmcs_ws/src/arm_description/urdf/arm_description.urdf (robot description, URDF)
Before this commit: robot arm_description, 7 links, 6 joints
Links:
- link link_2: mass 0.396 -> 0.356
- link link_3: mass 0.207 -> 0.107
- link link_4: mass 0.371 -> 0.351
- link link_5: mass 0.137 -> 0.150
- link link_6: mass 0.185 -> 0.300

Commit message: 111

File: rmcs_ws/src/arm_description/urdf/arm_description.urdf (robot description, URDF)
Before this commit: robot arm_description, 7 links, 6 joints
Links:
- link link_2: mass 0.356 -> 0.106
- link link_3: mass 0.107 -> 0.257
- link link_4: mass 0.351 -> 0.701
- link link_5: mass 0.150 -> 0.200
- link link_6: mass 0.300 -> 0.600

Commit message: 11

File: rmcs_ws/src/arm_description/urdf/arm_description.urdf (robot description, URDF)
Before this commit: robot arm_description, 7 links, 6 joints
Links:
- link link_5: mass 0.200 -> 0.100
- link link_6: mass 0.600 -> 0.300

Commit message: 222

File: rmcs_ws/src/arm_description/urdf/arm_description.urdf (robot description, URDF)
Before this commit: robot arm_description, 7 links, 6 joints
Joints:
- joint joint_2: limit lower=-1.084 upper=1.426 effort=63 velocity=4.71 -> lower=-1.084 upper=1.528 effort=63 velocity=4.71
- joint joint_3: limit lower=-1.36217 upper=0.5335 effort=35 velocity=4.71 -> lower=-1.37217 upper=0.5335 effort=35 velocity=4.71
- joint joint_4: limit lower=-3.14 upper=3.14 effort=18 velocity=7.54 -> lower=-3.1415926 upper=3.1415926 effort=18 velocity=7.54
- joint joint_5: limit lower=-1.74 upper=1.74 effort=6 velocity=24.61 -> lower=-1.967 upper=1.917 effort=6 velocity=24.61
- joint joint_6: limit lower=-3.14 upper=3.14 effort=3 velocity=10 -> lower=-3.1415926 upper=3.1415926 effort=3 velocity=10

Commit message: storage mine

File: rmcs_ws/src/arm_description/urdf/arm_description.urdf (robot description, URDF)
Before this commit: robot arm_description, 7 links, 6 joints
Joints:
- joint joint_3: limit lower=-1.37217 upper=0.5335 effort=35 velocity=4.71 -> lower=-1.450 upper=0.5335 effort=35 velocity=4.71

Commit message: feat:successfully run custome controller

File: rmcs_ws/src/arm_description/urdf/arm_description.urdf (robot description, URDF)
Before this commit: robot arm_description, 7 links, 6 joints
Links:
- link link_2: mass 0.106 -> 0.906
- link link_3: mass 0.257 -> 0.557
- link link_4: mass 0.701 -> 1.101
- link link_6: mass 0.300 -> 0.200

Commit message: Refactor stair control and arm target planning

File: rmcs_ws/src/arm_description/urdf/arm_description.urdf (robot description, URDF)
Before this commit: robot arm_description, 7 links, 6 joints
Joints:
- joint joint_5: limit lower=-1.967 upper=1.917 effort=6 velocity=24.61 -> lower=-1.967 upper=1.937 effort=6 velocity=24.61
