Commit message: refactor(lunar_rover):image_transmission change to uart instead of ttl
refactor(lunar_rover):image_transmission change to uart instead of ttl

refactor(lunar_rover):image_transmission change to uart instead of ttl

File: rmcs_ws/src/arm_description/urdf/arm_description.urdf (robot description, URDF)
Before this commit: robot arm_description, 7 links, 6 joints
Joints:
- joint joint_3: limit lower=-1.450 upper=0.5335 effort=35 velocity=4.71 -> lower=-1.57 upper=0.5335 effort=35 velocity=4.71

Commit message: feat(collision):added collision detection

File: rmcs_ws/src/arm_description/urdf/arm_description.urdf (robot description, URDF)
Before this commit: robot arm_description, 7 links, 6 joints
Links:
- link link_1: geometry visual mesh filename=package://arm_description/meshes/link_1.STL

Commit message: fix(arm_controller):fixed the blocking issue caused by the incorrect position of collision_apply().verified the feasibility of the new algorithm

File: rmcs_ws/src/arm_description/urdf/arm_description.urdf (robot description, URDF)
Before this commit: robot arm_description, 7 links, 6 joints
Links:
- link link_1: geometry collision mesh filename=package://arm_description/meshes/link_1.STL; visual mesh filename=package://arm_description/meshes/link_1.STL
